File: hardware/MCU_Power.kicad_sch (KiCad schematic)
At the start: 16 parts, among them U1 ISL854102FRZ-T

Commit message: wire up altimeter, temp, barometer, imu, gps to MCU
Parts:
- added C40: 2.2 uf, symbol Device:C_Small
- added C41: 1uf, symbol Device:C_Small
- added IC5: LDFPVR, SON65P200X200X100-7N-D, symbol Loaded_Libraries:LDFPVR
- added R79: 30.1k, symbol Device:R
- added R80: 10k, symbol Device:R
Connections:
- net +5V: now also C41.1, IC5.5 (EN), IC5.6 (VIN)
- net GND: now also C40.1, C41.2, IC5.4 (GND_1), IC5.7 (GND_2), R80.2
- new net: IC5.2 (ADJ/NC), R79.2, R80.1
- new net +3V3: C40.2, IC5.1 (VOUT), R79.1
Other:
- note added: "3.3V regulator"
- moved on the sheet: C11, C12, C13, C14, C15, C23, C24, C25, D1, D2, D3, L1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

Commit message: fixed electrical rules
Connections:
- no-connect marks 1 -> 2
Changed lines of the file:
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@@
+	)
+	(no_connect
+		(at 55.88 154.94)
 	)
 	(no_connect
