File: hardware/mcu.kicad_sch (KiCad schematic)
At the start: 27 parts, among them IC1 R7FA4M1AB3CFM#AA0

Commit message: fixed electrical rules
Parts:
- added JP15, JP16: SolderJumper_2_Open, symbol Jumper:SolderJumper_2_Open
- added JP20: SolderJumper_2_Bridged, symbol Jumper:SolderJumper_2_Bridged
Connections:
- net CS_1: now also JP15.1 (A)
- net IMU_SCK: now also JP20.2 (B)
- net SCK_MAG: now also JP16.1 (A)
- net SDA_MAG: now also JP15.2 (B)
- net DI2 renamed WAKE_ON_MOTION
- new net SCL/SPI_SLK : JP16.2 (B), JP20.1 (A)
Other:
- note added: "MCU SPI"
- note removed: "SPI"
- moved on the sheet: SCL1, SDA1
